File: CAD/CAN Board.kicad_pcb (KiCad board)
At the start: 4 copper layers, 35 x 50 mm, 100 parts, among them J1 Conn_01x04, J10 Conn_01x03, J11 Conn_01x03, J2 Conn_01x06, J3 USB_C_Receptacle_USB2.0_16P, J4 Conn_01x02, J5 Conn_01x02, J6 Conn_01x02, J7 Conn_01x02, J8 Conn_01x02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

Commit message: updated baord
Parts:
- C1, C2: value 27p -> 15p
- C18, C19, C25, C26, C32, C33, C39, C40, C46, C47, C53, C54: value 11.5p -> 18p
- Y1: value Crystal_GND24 -> 12MHz
- Y2, Y3, Y4, Y5, Y6, Y7: value Crystal_GND24 -> 40MHz
Other:
- board text added: "+|G|T|R|S|C"
- board text added: "CAN 1 H | L"
- board text added: "CAN 2"
- board text added: "CAN 3"
- board text added: "CAN 4"
- board text added: "CAN 5"
- board text added: "CAN 6"
- board text added: "C|G|D"
- board text added: "G|26|27|15"
- board text added: "G|T|R"
Changed lines of the file:
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@@
 			(drillshape 0)
 			(scaleselection 1)
-			(outputdirectory "Output/")
+			(outputdirectory "Fab/Gerber")
 		)
 	)
@@
 			)
 		)
-		(property "Value" "Crystal_GND24"
+		(property "Value" "40MHz"
 			(at 0 2.45 0)
 			(layer "F.Fab")
@@
 			)
 		)
-		(property "Datasheet" ""
+		(property "Datasheet" "ABM8G-40.000MHZ-18-D2Y-T"
 			(at 0 0 0)
 			(unlocked yes)
@@
 			)
 		)
-		(property "Value" "11.5p"
+		(property "Value" "18p"
 			(at 0 1.43 0)
 			(layer "F.Fab")
@@
 			)
 		)
-		(property "Value" "Crystal_GND24"
+		(property "Value" "12MHz"
 			(at 0 2.45 0)
 			(layer "F.Fab")
@@
 			)
 		)
-		(property "Datasheet" ""
+		(property "Datasheet" "Abracon ABM8-272-T3"
 			(at 0 0 0)
 			(unlocked yes)
@@
 			)
 		)
-		(property "Value" "11.5p"
+		(property "Value" "18p"
 			(at 0 1.43 0)
 			(layer "F.Fab")
@@
 			)
 		)
-		(property "Value" "11.5p"
+		(property "Value" "18p"
 			(at 0 1.43 0)
 			(layer "F.Fab")
@@
 			)
 		)
-		(property "Value" "11.5p"
+		(property "Value" "18p"
 			(at 0 1.43 0)
 			(layer "F.Fab")
@@
 			)
 		)
-		(property "Value" "11.5p"
+		(property "Value" "18p"
 			(at 0 1.43 0)
 			(layer "F.Fab")
@@
 			)
 		)
-		(property "Value" "Crystal_GND24"
+		(property "Value" "40MHz"
 			(at 0 2.45 0)
 			(layer "F.Fab")
@@
 			)
 		)
-		(property "Datasheet" ""
+		(property "Datasheet" "ABM8G-40.000MHZ-18-D2Y-T"
 			(at 0 0 0)
 			(unlocked yes)
@@
 			)
 		)
-		(property "Value" "11.5p"
+		(property "Value" "18p"
 			(at 0 1.43 0)
 			(layer "F.Fab")
@@
 			)
 		)
-		(property "Value" "11.5p"
+		(property "Value" "18p"
 			(at 0 1.43 0)
 			(layer "F.Fab")
@@
 			)
 		)
-		(property "Value" "Crystal_GND24"
+		(property "Value" "40MHz"
 			(at 0 2.45 0)
 			(layer "F.Fab")
@@
 			)
 		)
-		(property "Datasheet" ""
+		(property "Datasheet" "ABM8G-40.000MHZ-18-D2Y-T"
 			(at 0 0 0)
 			(unlocked yes)
@@
 			)
 		)
-		(property "Value" "Crystal_GND24"
+		(property "Value" "40MHz"
 			(at 0 2.45 0)
 			(layer "F.Fab")
@@
 			)
 		)
-		(property "Datasheet" ""
+		(property "Datasheet" "ABM8G-40.000MHZ-18-D2Y-T"
 			(at 0 0 0)
 			(unlocked yes)
@@
 			)
 		)
-		(property "Value" "11.5p"
+		(property "Value" "18p"
 			(at 0 1.43 0)
 			(layer "F.Fab")
@@
 			)
 		)
-		(property "Value" "11.5p"
+		(property "Value" "18p"
 			(at 0 1.43 0)
 			(layer "F.Fab")
@@
 			)
 		)
-		(property "Value" "11.5p"
+		(property "Value" "18p"
 			(at 0 1.43 0)
 			(layer "F.Fab")
@@
 			)
 		)
-		(property "Value" "27p"
+		(property "Value" "15p"
 			(at 0 1.43 0)
 			(layer "F.Fab")
@@
 			)
 		)
-		(property "Value" "Crystal_GND24"
+		(property "Value" "40MHz"
 			(at 0 2.45 0)
 			(layer "F.Fab")
@@
 			)
 		)
-		(property "Datasheet" ""
+		(property "Datasheet" "ABM8G-40.000MHZ-18-D2Y-T"
 			(at 0 0 0)
 			(unlocked yes)
@@
 			)
 		)
-		(property "Value" "11.5p"
+		(property "Value" "18p"
 			(at 0 1.43 0)
 			(layer "F.Fab")
@@
 			)
 		)
-		(property "Value" "27p"
+		(property "Value" "15p"
 			(at 0 1.43 0)
 			(layer "F.Fab")
@@
 			)
 		)
-		(property "Value" "11.5p"
+		(property "Value" "18p"
 			(at 0 1.43 0)
 			(layer "F.Fab")
@@
 			)
 		)
-		(property "Value" "Crystal_GND24"
+		(property "Value" "40MHz"
 			(at 0 2.45 0)
 			(layer "F.Fab")
@@
 			)
 		)
-		(property "Datasheet" ""
+		(property "Datasheet" "ABM8G-40.000MHZ-18-D2Y-T"
 			(at 0 0 0)
 			(unlocked yes)
@@
 		(layer "Edge.Cuts")
 	)
+	(gr_text "CAN 2"
+		(at 58.5 24.095 90)
+		(layer "B.SilkS")
+		(effects
+			(font
+				(size 0.8 0.8)
+				(thickness 0.15)
+				(bold yes)
+			)
+			(justify mirror)
+		)
+	)
 	(gr_text "BOOT"
-		(at 33 23 0)
+		(at 31.5 22.5 90)
 		(layer "B.SilkS")
 		(effects
@@
 				(bold yes)
 			)
-			(justify left bottom mirror)
+			(justify mirror)
 		)
 	)
 	(gr_text "RST"
-		(at 39.55 55.5 90)
+		(at 39.5 56.5 90)
 		(layer "B.SilkS")
 		(effects
@@
 				(bold yes)
 			)
-			(justify left bottom mirror)
+			(justify mirror)
 		)
 	)
-	(gr_text "GPIO"
-		(at 36 55 90)
+	(gr_text "CAN 5"
+		(at 58.5 49.895 90)
 		(layer "B.SilkS")
 		(effects
@@
 				(bold yes)
 			)
-			(justify left bottom mirror)
+			(justify mirror)
 		)
 	)
-	(gr_text "SWD"
-		(at 31.5 46 90)
+	(gr_text "G|T|R"
+		(at 31 39.5 90)
 		(layer "B.SilkS")
 		(effects
@@
 				(bold yes)
 			)
-			(justify left bottom mirror)
+			(justify mirror)
 		)
 	)
-	(gr_text "SPI"
-		(at 31.5 55.5 90)
+	(gr_text "CAN 1\nH | L"
+		(at 59 15.5 90)
 		(layer "B.SilkS")
 		(effects
@@
 				(bold yes)
 			)
-			(justify left bottom mirror)
+			(justify bottom mirror)
 		)
 	)
-	(gr_text "UART\n"
-		(at 31.5 38 90)
+	(gr_text "+|G|T|R|S|C"
+		(at 31 56.5 90)
 		(layer "B.SilkS")
 		(effects
@@
 				(bold yes)
 			)
-			(justify left bottom mirror)
+			(justify mirror)
+		)
+	)
+	(gr_text "CAN 3"
+		(at 58.5 32.695 90)
+		(layer "B.SilkS")
+		(effects
+			(font
+				(size 0.8 0.8)
+				(thickness 0.15)
+				(bold yes)
+			)
+			(justify mirror)
+		)
+	)
+	(gr_text "C|G|D"
+		(at 31 47 90)
+		(layer "B.SilkS")
+		(effects
+			(font
+				(size 0.8 0.8)
+				(thickness 0.15)
+				(bold yes)
+			)
+			(justify mirror)
+		)
+	)
+	(gr_text "CAN 6"
+		(at 58.5 58.495 90)
+		(layer "B.SilkS")
+		(effects
+			(font
+				(size 0.8 0.8)
+				(thickness 0.15)
+				(bold yes)
+			)
+			(justify mirror)
+		)
+	)
+	(gr_text "CAN 4"
+		(at 58.5 41.295 90)
+		(layer "B.SilkS")
+		(effects
+			(font
+				(size 0.8 0.8)
+				(thickness 0.15)
+				(bold yes)
+			)
+			(justify mirror)
+		)
+	)
+	(gr_text "G|26|27|15"
+		(at 36 57.75 90)
+		(layer "B.SilkS")
+		(effects
+			(font
+				(size 0.8 0.8)
+				(thickness 0.15)
+				(bold yes)
+			)
+			(justify mirror)
+		)
+	)
+	(gr_text "SPI"
+		(at 32 56.5 270)
+		(layer "F.SilkS")
+		(effects
+			(font
+				(size 0.8 0.8)
+				(thickness 0.15)
+				(bold yes)
+			)
+		)
+	)
+	(gr_text "SWD"
+		(at 32 47 270)
+		(layer "F.SilkS")
+		(effects
+			(font
+				(size 0.8 0.8)
+				(thickness 0.15)
+				(bold yes)
+			)
+		)
+	)
+	(gr_text "UART\n"
+		(at 32 42 270)
+		(layer "F.SilkS")
+		(effects
+			(font
+				(size 0.8 0.8)
+				(thickness 0.15)
+				(bold yes)
+			)
+		)
+	)
+	(gr_text "GPIO"
+		(at 37 57.75 270)
+		(layer "F.SilkS")
+		(effects
+			(font
+				(size 0.8 0.8)
+				(thickness 0.15)
+				(bold yes)
+			)
 		)
 	)

Commit message: added LED and cleanup
Parts:
- added D1: LED, LED_SMD:LED_0603_1608Metric_Pad1.05x0.95mm_HandSolder, F.Cu at (39.0, 50.0)
- added J12: Conn_01x03, Connector_Molex:Molex_PicoBlade_53047-0310_1x03_P1.25mm_Vertical, F.Cu at (29.1, 37.8)
- added Q1: NMOS, Package_TO_SOT_SMD:SOT-323_SC-70, F.Cu at (35.5, 52.0)
- added R19: 1k, Resistor_SMD:R_0603_1608Metric_Pad0.98x0.95mm_HandSolder, F.Cu at (39.0, 51.5)
- J1: value Conn_01x04 -> Conn_01x03; footprint Connector_Molex:Molex_PicoBlade_53047-0410_1x04_P1.25mm_Vertical -> Connector_Molex:Molex_PicoBlade_53047-0310_1x03_P1.25mm_Vertical
- J10: value Conn_01x03 -> Conn_01x02; footprint Connector_Molex:Molex_PicoBlade_53047-0310_1x03_P1.25mm_Vertical -> Connector_Molex:Molex_PicoBlade_53047-0210_1x02_P1.25mm_Vertical
- J2: value Conn_01x06 -> Conn_01x04; footprint Connector_Molex:Molex_PicoBlade_53047-0610_1x06_P1.25mm_Vertical -> Connector_Molex:Molex_PicoBlade_53047-0410_1x04_P1.25mm_Vertical
- moved J10 6.25 mm to (29.1, 44.5)
- moved J2 5.94 mm to (34.5, 55.6)
- moved J1 5.08 mm to (29.1, 56.8)
- moved J11 4.25 mm to (29.1, 50.0)
- moved SW1 0.71 mm to (40.0, 53.8)
Connections:
- J1 pad 1: GND -> GPIO 15
- J10 pad 1: GND -> TX0
- J10 pad 2: TX0 -> RX0
- J2 pad 1: +5V -> SPI1 TX
- J2 pad 2: GND -> SPI1 RX
- J2 pad 3: SPI1 TX -> SPI1 CSn
- J2 pad 4: SPI1 RX -> SPI1 SCK
Routing:
- net GPIO 15: track 24.6 -> 33.4 mm
- net RX0: track 8.16 -> 13.6 mm
- net TX0: track 7.55 -> 12.6 mm
- net +3V3: track 132.2 -> 135.9 mm
- net Net-(Q1-D): track 0.00 -> 3.65 mm
- net ADC 0: track 24.4 -> 27.3 mm
- net SWD: track 18.6 -> 15.9 mm
- net ADC 1: track 27.1 -> 29.6 mm
- net RUN: track 15.4 -> 17.0 mm
- net Net-(D1-K): track 0.00 -> 1.52 mm
- net GND: track 209.7 -> 210.8 mm, vias 31 -> 32
- net SPI1 SCK: track 22.0 -> 21.1 mm
- net SWCLK: track 14.3 -> 15.1 mm
- net SPI1 CSn: track 20.3 -> 19.7 mm
Other:
- outline, holes or cut-outs redrawn
- board text added: "15|26|27"
- board text added: "5|3.3|G"
- board text added: "PWR|UART|SWD"
- board text added: "TX|RX"
- board text added: "TX|RX|S|C"
- board text removed: "+|G|T|R|S|C"
- board text removed: "G|26|27|15"
- board text removed: "G|T|R"
- board text removed: "SWD"
- board text removed: "UART"
