File: CAD/CAN Board.kicad_pcb (KiCad board)
At the start: 4 copper layers, 35 x 50 mm, 104 parts, among them J1 Conn_01x03, J10 Conn_01x02, J11 Conn_01x03, J12 Conn_01x03, J2 Conn_01x04, J3 USB_C_Receptacle_USB2.0_16P, J4 Conn_01x02, J5 Conn_01x02, J6 Conn_01x02, J7 Conn_01x02, J8 Conn_01x02, J9 Conn_01x02, Q1 NMOS, SW1 SW_Push, SW2 SW_Push, U1 RP2040, U2 W25Q128JVS, U3 MIC5504-3.3YM5, U4 MCP251863T-E/9PX, U5 MCP251863T-E/9PX, U6 MCP251863T-E/9PX, U7 MCP251863T-E/9PX, U8 MCP251863T-E/9PX, U9 MCP251863T-E/9PX, Y1 12MHz, Y2 40MHz, Y3 40MHz, Y4 40MHz, Y5 40MHz, Y6 40MHz, Y7 40MHz

Commit message: added screw holes
Parts:
- added REF**: MountingHole_2.2mm_M2, MountingHole:MountingHole_2.2mm_M2, F.Cu at (59.0, 9.00)
- added REF**: MountingHole_2.2mm_M2, MountingHole:MountingHole_2.2mm_M2, F.Cu at (30.0, 65.0)
- added REF**: MountingHole_2.2mm_M2, MountingHole:MountingHole_2.2mm_M2, F.Cu at (59.0, 65.0)
Routing:
- net GND: track 210.8 -> 196.1 mm, vias 32 -> 40
- added copper zone on F.Cu, net GND
Other:
- board size 35 x 50 mm -> 35 x 62 mm

Commit message: updated board
Parts:
- added R20: 220, Resistor_SMD:R_0603_1608Metric_Pad0.98x0.95mm_HandSolder, F.Cu at (33.0, 51.9)
Connections:
- Q1 pad 2: GPIO 15 -> Net-(Q1-G)
- U4 pad 29: unconnected-(U4-EP-Pad29) -> GND
- U4 pad 8: CAN1 INT1 -> unconnected-(U4-nINT1/GPIO1-Pad8)
- U4 pad 9: unconnected-(U4-nINT0/GPIO0/XSTBY-Pad9) -> CAN1 INT1
- U5 pad 29: unconnected-(U5-EP-Pad29) -> GND
- U5 pad 8: CAN2 INT1 -> unconnected-(U5-nINT1/GPIO1-Pad8)
- U5 pad 9: unconnected-(U5-nINT0/GPIO0/XSTBY-Pad9) -> CAN2 INT1
- U6 pad 29: unconnected-(U6-EP-Pad29) -> GND
- U6 pad 8: CAN3 INT1 -> unconnected-(U6-nINT1/GPIO1-Pad8)
- U6 pad 9: unconnected-(U6-nINT0/GPIO0/XSTBY-Pad9) -> CAN3 INT1
- U7 pad 29: unconnected-(U7-EP-Pad29) -> GND
- U7 pad 8: CAN4 INT1 -> unconnected-(U7-nINT1/GPIO1-Pad8)
- U7 pad 9: unconnected-(U7-nINT0/GPIO0/XSTBY-Pad9) -> CAN4 INT1
- U8 pad 29: unconnected-(U8-EP-Pad29) -> GND
- U8 pad 8: CAN5 INT1 -> unconnected-(U8-nINT1/GPIO1-Pad8)
- U8 pad 9: unconnected-(U8-nINT0/GPIO0/XSTBY-Pad9) -> CAN5 INT1
- U9 pad 29: unconnected-(U9-EP-Pad29) -> GND
- U9 pad 8: CAN6 INT1 -> unconnected-(U9-nINT1/GPIO1-Pad8)
- U9 pad 9: unconnected-(U9-nINT0/GPIO0/XSTBY-Pad9) -> CAN6 INT1
Routing:
- net +5V: track 55.7 -> 86.6 mm
- net GND: track 196.1 -> 219.5 mm, vias 40 -> 34
- net SPI0 1CS: track 37.2 -> 34.6 mm
- net Net-(Q1-G): track 0.00 -> 2.27 mm
- net SPI0 6CS: track 31.1 -> 28.9 mm
- net SPI0 5CS: track 27.5 -> 25.7 mm
- net GPIO 15: track 33.4 -> 31.8 mm
- net CAN6 INT1: track 29.2 -> 30.3 mm
- net SPI0 3CS: track 28.0 -> 27.0 mm
- net CAN4 INT1: track 14.7 -> 15.5 mm
- net CAN3 INT1: track 12.1 -> 12.9 mm
- net CAN2 INT1: track 19.4 -> 20.1 mm
- net CAN5 INT1: track 21.6 -> 22.4 mm
- net CAN1 INT1: track 25.3 -> 26.1 mm
- net Net-(U9-RXCAN): track 9.80 -> 9.21 mm
