File: CAD/CAN Board.kicad_pcb (KiCad board)
At the start: 4 copper layers, 35 x 62 mm, 108 parts, among them J1 Conn_01x03, J10 Conn_01x02, J11 Conn_01x03, J12 Conn_01x03, J2 Conn_01x04, J3 USB_C_Receptacle_USB2.0_16P, J4 Conn_01x02, J5 Conn_01x02, J6 Conn_01x02, J7 Conn_01x02, J8 Conn_01x02, J9 Conn_01x02, Q1 NMOS, SW1 SW_Push, SW2 SW_Push, U1 RP2040, U2 W25Q128JVS, U3 MIC5504-3.3YM5, U4 MCP251863T-E/9PX, U5 MCP251863T-E/9PX, U6 MCP251863T-E/9PX, U7 MCP251863T-E/9PX, U8 MCP251863T-E/9PX, U9 MCP251863T-E/9PX, Y1 12MHz, Y2 40MHz, Y3 40MHz, Y4 40MHz, Y5 40MHz, Y6 40MHz, Y7 40MHz

Commit message: updated CAN termination
Parts:
- removed C23, C30, C37, C44, C51, C58: 560p, Capacitor_SMD:C_0603_1608Metric
- removed R20: 220, Resistor_SMD:R_0603_1608Metric_Pad0.98x0.95mm_HandSolder
- C22, C29, C36, C43, C50, C57: value 560p -> 4.7n
- R10, R11, R12, R13, R14, R15, R16, R17, R18, R7, R8, R9: value 100 -> 60
- R19: footprint Resistor_SMD:R_0603_1608Metric_Pad0.98x0.95mm_HandSolder -> Resistor_SMD:R_0603_1608Metric
- moved C57 4.00 mm to (57.0, 55.5)
- moved R8 4.00 mm to (57.0, 17.0)
- moved C50 3.50 mm to (57.0, 47.5)
- moved R10 3.50 mm to (57.0, 25.0)
- moved C43 3.00 mm to (57.0, 39.5)
- moved R12 3.00 mm to (57.0, 33.0)
- moved R17 2.50 mm to (57.0, 58.5)
- moved C36 2.00 mm to (57.0, 31.5)
- moved R14 2.00 mm to (57.0, 41.0)
- moved R15 2.00 mm to (57.0, 50.5)
- moved J4 1.53 mm to (60.5, 15.8)
- moved C29 1.50 mm to (57.0, 23.5)
- moved R13 1.50 mm to (57.0, 42.5)
- moved R16 1.50 mm to (57.0, 49.0)
- moved J9 1.48 mm to (60.5, 55.8)
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Connections:
- Q1 pad 2: Net-(Q1-G) -> GPIO 15
- R10 pad 2: Net-(C30-Pad1) -> Net-(C29-Pad1)
- R12 pad 2: Net-(C37-Pad1) -> Net-(C36-Pad1)
- R14 pad 2: Net-(C44-Pad1) -> Net-(C43-Pad1)
- R16 pad 2: Net-(C51-Pad1) -> Net-(C50-Pad1)
- R18 pad 2: Net-(C58-Pad1) -> Net-(C57-Pad1)
- R8 pad 2: Net-(C23-Pad1) -> Net-(C22-Pad1)
Routing:
- net GND: track 219.5 -> 202.9 mm, vias 34 -> 31
- net CAN6H: track 13.6 -> 8.55 mm
- net CAN5H: track 12.8 -> 8.52 mm
- net CAN4H: track 12.3 -> 8.52 mm
- net CAN6L: track 10.1 -> 7.22 mm
- net CAN3H: track 11.2 -> 8.39 mm
- net CAN1H: track 11.0 -> 8.55 mm
- net CAN2H: track 10.9 -> 8.52 mm
- net Net-(Q1-G): track 2.27 -> 0.00 mm
- net CAN5L: track 9.45 -> 7.20 mm
- net RUN: track 17.0 -> 15.2 mm
- net CAN4L: track 9.02 -> 7.20 mm
- net Net-(C30-Pad1): track 1.59 -> 0.00 mm
- net Net-(C23-Pad1): track 1.59 -> 0.00 mm
- net Net-(C37-Pad1): track 1.59 -> 0.00 mm
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
Commit message: updated code
Other:
- board text added: "H | L CAN 1"
- board text removed: "CAN 1 H | L"
